File: CRServoF_WLCSP36.sch (KiCad schematic (older format))
At the start: 33 parts, among them J1 Conn_02x06_Counter_Clockwise, J2 Conn_02x06_Counter_Clockwise, J3 Conn_01x03, J4 Conn_01x04, J5 Conn_01x03, U1 TPS727xxDSE, U2 STM32F051T8Yx

Commit message: update schematic and silk screen
Parts:
- U1: value TPS727xxDSE -> TPS72733DSE
Changed lines of the file:
@@
 P 2700 1900
 F 0 "U1" H 2700 2365 50  0000 C CNN
-F 1 "TPS727xxDSE" H 2700 2274 50  0000 C CNN
+F 1 "TPS72733DSE" H 2700 2274 50  0000 C CNN
 F 2 "Package_SON:WSON-6_1.5x1.5mm_P0.5mm" H 2700 1900 50  0001 C CNN
 F 3 "" H 2700 1900 50  0001 C CNN
